Commit message: reduce damping

File: double_pendulum_description/urdf/double_pendulum.xacro (robot description, xacro)
@@ -50,5 +50,5 @@
     <origin xyz="0 ${width} ${height1 - axel_offset}" rpy="0 0 0"/>
     <axis xyz="0 1 0"/>
-    <dynamics damping="0.7"/>
+    <dynamics damping="0.1"/>
   </joint>
   <!-- Middle Link -->
@@ -81,5 +81,5 @@
     <origin xyz="0 ${width} ${height2 - axel_offset*2}" rpy="0 0 0"/>
     <axis xyz="0 1 0"/>
-    <dynamics damping="0.7"/>
+    <dynamics damping="0.1"/>
   </joint>
   <!-- Top Link -->

Commit message: basic setup complete

File: double_pendulum_description/urdf/double_pendulum.xacro (robot description, xacro)
@@ -1,4 +1,4 @@
 <?xml version="1.0"?>
-<!-- Revolute-Revolute Manipulator -->
+<!-- Balancing Double Pendulum -->
 <robot name="double_pendulum" xmlns:xacro="http://www.ros.org/wiki/xacro">
   <!-- Constants for robot dimensions -->
@@ -6,18 +6,49 @@
   <xacro:property name="mass" value="1" /> <!-- arbitrary value for mass -->
   <xacro:property name="width" value="0.1" /> <!-- Square dimensions (widthxwidth) of beams -->
-  <xacro:property name="height1" value="2" /> <!-- Link 1 -->
+  <xacro:property name="height1" value="0.2" /> <!-- Link 1 -->
   <xacro:property name="height2" value="1" /> <!-- Link 2 -->
   <xacro:property name="height3" value="1" /> <!-- Link 3 -->
-  <xacro:property name="camera_link" value="0.05" /> <!-- Size of square 'camera' box -->
-  <xacro:property name="axel_offset" value="0.05" /> <!-- Space btw top of beam and the each joint -->
+  <xacro:property name="foot_height" value="0.1" /> <!-- Foot dimensions -->
+  <xacro:property name="foot_width" value="0.5" />
+  <xacro:property name="axel_offset" value="0.05" /> <!-- How far keep joints away from each other -->
   <!-- Import all Gazebo-customization elements, including Gazebo colors -->
   <xacro:include filename="$(find double_pendulum_description)/urdf/double_pendulum.gazebo" />
   <!-- Import Rviz colors -->
   <xacro:include filename="$(find double_pendulum_description)/urdf/materials.xacro" />
-  <!-- Used for fixing robot to Gazebo 'base_link' -->
-  <link name="world"/>
+  <!-- Used for fixing robot foot to the world -->
+  <!--<link name="world"/>
   <joint name="fixed" type="fixed">
     <parent link="world"/>
+    <child link="foot"/>
+  </joint>-->
+  <!-- Foot Link-->
+  <link name="foot">
+    <collision>
+      <origin xyz="0 0 ${foot_height/2}" rpy="0 0 0"/>
+      <geometry>
+        <box size="${foot_width} ${foot_width} ${foot_height}"/>
+      </geometry>
+    </collision>
+    <visual>
+      <origin xyz="0 0 ${foot_height/2}" rpy="0 0 0"/>
+      <geometry>
+        <box size="${foot_width} ${foot_width} ${foot_height}"/>
+      </geometry>
+      <material name="grey"/>
+    </visual>
+    <inertial>
+      <origin xyz="0 0 ${foot_height/2}" rpy="0 0 0"/>
+      <mass value="${mass}"/>
+      <inertia
+        ixx="${mass / 12.0 * (foot_width*foot_width + foot_height*foot_height)}" ixy="0.0" ixz="0.0"
+        iyy="${mass / 12.0 * (foot_height*foot_height + foot_width*foot_width)}" iyz="0.0"
+        izz="${mass / 12.0 * (foot_width*foot_width + foot_width*foot_width)}"/>
+    </inertial>
+  </link>
+  <joint name="foot_joint" type="fixed">
+    <parent link="foot"/>
     <child link="link1"/>
+    <origin xyz="0 0 ${foot_height}" rpy="0 0 0"/>
+    <axis xyz="0 1 0"/>
   </joint>
   <!-- Base Link -->
@@ -26,5 +57,5 @@
       <origin xyz="0 0 ${height1/2}" rpy="0 0 0"/>
       <geometry>
-	<box size="${width} ${width} ${height1}"/>
+        <box size="${width} ${width} ${height1}"/>
       </geometry>
     </collision>
@@ -32,7 +63,7 @@
       <origin xyz="0 0 ${height1/2}" rpy="0 0 0"/>
       <geometry>
-	<box size="${width} ${width} ${height1}"/>
+        <box size="${width} ${width} ${height1}"/>
       </geometry>
-      <material name="orange"/>
+      <material name="grey"/>
     </visual>
     <inertial>
@@ -40,7 +71,7 @@
       <mass value="${mass}"/>
       <inertia
-	  ixx="${mass / 12.0 * (width*width + height1*height1)}" ixy="0.0" ixz="0.0"
-	  iyy="${mass / 12.0 * (height1*height1 + width*width)}" iyz="0.0"
-	  izz="${mass / 12.0 * (width*width + width*width)}"/>
+        ixx="${mass / 12.0 * (width*width + height1*height1)}" ixy="0.0" ixz="0.0"
+        iyy="${mass / 12.0 * (height1*height1 + width*width)}" iyz="0.0"
+        izz="${mass / 12.0 * (width*width + width*width)}"/>
     </inertial>
   </link>
@@ -57,5 +88,5 @@
       <origin xyz="0 0 ${height2/2 - axel_offset}" rpy="0 0 0"/>
       <geometry>
-	<box size="${width} ${width} ${height2}"/>
+        <box size="${width} ${width} ${height2}"/>
       </geometry>
     </collision>
@@ -63,7 +94,7 @@
       <origin xyz="0 0 ${height2/2 - axel_offset}" rpy="0 0 0"/>
       <geometry>
-	<box size="${width} ${width} ${height2}"/>
+        <box size="${width} ${width} ${height2}"/>
       </geometry>
-      <material name="black"/>
+      <material name="red"/>
     </visual>
     <inertial>
@@ -71,7 +102,7 @@
       <mass value="${mass}"/>
       <inertia
-	  ixx="${mass / 12.0 * (width*width + height2*height2)}" ixy="0.0" ixz="0.0"
-	  iyy="${mass / 12.0 * (height2*height2 + width*width)}" iyz="0.0"
-	  izz="${mass / 12.0 * (width*width + width*width)}"/>
+        ixx="${mass / 12.0 * (width*width + height2*height2)}" ixy="0.0" ixz="0.0"
+        iyy="${mass / 12.0 * (height2*height2 + width*width)}" iyz="0.0"
+        izz="${mass / 12.0 * (width*width + width*width)}"/>
     </inertial>
   </link>
@@ -88,5 +119,5 @@
       <origin xyz="0 0 ${height3/2 - axel_offset}" rpy="0 0 0"/>
       <geometry>
-	<box size="${width} ${width} ${height3}"/>
+        <box size="${width} ${width} ${height3}"/>
       </geometry>
     </collision>
@@ -94,7 +125,7 @@
       <origin xyz="0 0 ${height3/2 - axel_offset}" rpy="0 0 0"/>
       <geometry>
-	<box size="${width} ${width} ${height3}"/>
+        <box size="${width} ${width} ${height3}"/>
       </geometry>
-      <material name="orange"/>
+      <material name="red"/>
     </visual>
     <inertial>
@@ -102,73 +133,10 @@
       <mass value="${mass}"/>
       <inertia
-	  ixx="${mass / 12.0 * (width*width + height3*height3)}" ixy="0.0" ixz="0.0"
-	  iyy="${mass / 12.0 * (height3*height3 + width*width)}" iyz="0.0"
-	  izz="${mass / 12.0 * (width*width + width*width)}"/>
+        ixx="${mass / 12.0 * (width*width + height3*height3)}" ixy="0.0" ixz="0.0"
+        iyy="${mass / 12.0 * (height3*height3 + width*width)}" iyz="0.0"
+        izz="${mass / 12.0 * (width*width + width*width)}"/>
     </inertial>
   </link>
-  <joint name="hokuyo_joint" type="fixed">
-    <axis xyz="0 1 0" />
-    <origin xyz="0 0 ${height3 - axel_offset/2}" rpy="0 0 0"/>
-    <parent link="link3"/>
-    <child link="hokuyo_link"/>
-  </joint>
-  <!-- Hokuyo Laser -->
-  <link name="hokuyo_link">
-    <collision>
-      <origin xyz="0 0 0" rpy="0 0 0"/>
-      <geometry>
-	<box size="0.1 0.1 0.1"/>
-      </geometry>
-    </collision>
-    <visual>
-      <origin xyz="0 0 0" rpy="0 0 0"/>
-      <geometry>
-        <mesh filename="package://double_pendulum_description/meshes/hokuyo.dae"/>
-      </geometry>
-    </visual>
-    <inertial>
-      <mass value="1e-5" />
-      <origin xyz="0 0 0" rpy="0 0 0"/>
-      <inertia ixx="1e-6" ixy="0" ixz="0" iyy="1e-6" iyz="0" izz="1e-6" />
-    </inertial>
-  </link>
-  <joint name="camera_joint" type="fixed">
-    <axis xyz="0 1 0" />
-    <origin xyz="${camera_link} 0 ${height3 - axel_offset*2}" rpy="0 0 0"/>
-    <parent link="link3"/>
-    <child link="camera_link"/>
-  </joint>
-  <!-- Camera -->
-  <link name="camera_link">
-    <collision>
-      <origin xyz="0 0 0" rpy="0 0 0"/>
-      <geometry>
-	<box size="${camera_link} ${camera_link} ${camera_link}"/>
-      </geometry>
-    </collision>
-    <visual>
-      <origin xyz="0 0 0" rpy="0 0 0"/>
-      <geometry>
-	<box size="${camera_link} ${camera_link} ${camera_link}"/>
-      </geometry>
-      <material name="red"/>
-    </visual>
-    <inertial>
-      <mass value="1e-5" />
-      <origin xyz="0 0 0" rpy="0 0 0"/>
-      <inertia ixx="1e-6" ixy="0" ixz="0" iyy="1e-6" iyz="0" izz="1e-6" />
-    </inertial>
-  </link>
-  <!-- generate an optical frame http://www.ros.org/reps/rep-0103.html#suffix-frames
-      so that ros and opencv can operate on the camera frame correctly -->
-  <joint name="camera_optical_joint" type="fixed">
-    <!-- these values have to be these values otherwise the gazebo camera image
-        won't be aligned properly with the frame it is supposedly originating from -->
-    <origin xyz="0 0 0" rpy="${-pi/2} 0 ${-pi/2}"/>
-    <parent link="camera_link"/>
-    <child link="camera_link_optical"/>
-  </joint>
-  <link name="camera_link_optical">
-  </link>
+  <!-- Motors so we can actuate the joints -->
   <transmission name="tran1">
     <type>transmission_interface/SimpleTransmission</type>

Commit message: small model tweaks

File: double_pendulum_description/urdf/double_pendulum.xacro (robot description, xacro)
@@ -9,5 +9,5 @@
   <xacro:property name="height2" value="1" /> <!-- Link 2 -->
   <xacro:property name="height3" value="1" /> <!-- Link 3 -->
-  <xacro:property name="foot_height" value="0.1" /> <!-- Foot dimensions -->
+  <xacro:property name="foot_height" value="0.05" /> <!-- Foot dimensions -->
   <xacro:property name="foot_width" value="0.5" />
   <xacro:property name="axel_offset" value="0.05" /> <!-- How far keep joints away from each other -->
@@ -49,5 +49,5 @@
     <parent link="foot"/>
     <child link="link1"/>
-    <origin xyz="0 0 ${foot_height}" rpy="0 0 0"/>
+    <origin xyz="0 -${width} ${foot_height}" rpy="0 0 0"/>
     <axis xyz="0 1 0"/>
   </joint>

Commit message: smooth balancing with extra damping via matlab

File: double_pendulum_description/urdf/double_pendulum.xacro (robot description, xacro)
@@ -4,9 +4,9 @@
   <!-- Constants for robot dimensions -->
   <xacro:property name="PI" value="3.1415926535897931"/>
-  <xacro:property name="mass" value="1" /> <!-- arbitrary value for mass -->
+  <xacro:property name="mass" value="1.0" /> <!-- arbitrary value for mass -->
   <xacro:property name="width" value="0.1" /> <!-- Square dimensions (widthxwidth) of beams -->
   <xacro:property name="height1" value="0.2" /> <!-- Link 1 -->
-  <xacro:property name="height2" value="1" /> <!-- Link 2 -->
-  <xacro:property name="height3" value="1" /> <!-- Link 3 -->
+  <xacro:property name="height2" value="1.1" /> <!-- Link 2 -->
+  <xacro:property name="height3" value="1.1" /> <!-- Link 3 -->
   <xacro:property name="foot_height" value="0.05" /> <!-- Foot dimensions -->
   <xacro:property name="foot_width" value="0.5" />
@@ -17,9 +17,9 @@
   <xacro:include filename="$(find double_pendulum_description)/urdf/materials.xacro" />
   <!-- Used for fixing robot foot to the world -->
-  <!--<link name="world"/>
+  <link name="world"/>
   <joint name="fixed" type="fixed">
     <parent link="world"/>
     <child link="foot"/>
-  </joint>-->
+  </joint>
   <!-- Foot Link-->
   <link name="foot">
@@ -40,5 +40,5 @@
       <origin xyz="0 0 ${foot_height/2}" rpy="0 0 0"/>
       <mass value="${mass}"/>
-      <inertia
+    <inertia
         ixx="${mass / 12.0 * (foot_width*foot_width + foot_height*foot_height)}" ixy="0.0" ixz="0.0"
         iyy="${mass / 12.0 * (foot_height*foot_height + foot_width*foot_width)}" iyz="0.0"
@@ -70,5 +70,5 @@
       <origin xyz="0 0 ${height1/2}" rpy="0 0 0"/>
       <mass value="${mass}"/>
-      <inertia
+    <inertia
         ixx="${mass / 12.0 * (width*width + height1*height1)}" ixy="0.0" ixz="0.0"
         iyy="${mass / 12.0 * (height1*height1 + width*width)}" iyz="0.0"
@@ -81,5 +81,5 @@
     <origin xyz="0 ${width} ${height1 - axel_offset}" rpy="0 0 0"/>
     <axis xyz="0 1 0"/>
-    <dynamics damping="0.1"/>
+    <dynamics damping="0.5"/>
   </joint>
   <!-- Middle Link -->
@@ -88,5 +88,5 @@
       <origin xyz="0 0 ${height2/2 - axel_offset}" rpy="0 0 0"/>
       <geometry>
-        <box size="${width} ${width} ${height2}"/>
+        <box size="${width} ${width} ${height2+axel_offset}"/>
       </geometry>
     </collision>
@@ -101,8 +101,9 @@
       <origin xyz="0 0 ${height2/2 - axel_offset}" rpy="0 0 0"/>
       <mass value="${mass}"/>
+      <!-- inertias copied from matlab model-->
       <inertia
-        ixx="${mass / 12.0 * (width*width + height2*height2)}" ixy="0.0" ixz="0.0"
-        iyy="${mass / 12.0 * (height2*height2 + width*width)}" iyz="0.0"
-        izz="${mass / 12.0 * (width*width + width*width)}"/>
+        ixx="0.3345833333333" ixy="0.0" ixz="0.0"
+        iyy="0.3345833333333" iyz="0.0"
+        izz="0.0025"/>
     </inertial>
   </link>
@@ -112,5 +113,5 @@
     <origin xyz="0 ${width} ${height2 - axel_offset*2}" rpy="0 0 0"/>
     <axis xyz="0 1 0"/>
-    <dynamics damping="0.1"/>
+    <dynamics damping="0.5"/>
   </joint>
   <!-- Top Link -->
@@ -133,7 +134,7 @@
       <mass value="${mass}"/>
       <inertia
-        ixx="${mass / 12.0 * (width*width + height3*height3)}" ixy="0.0" ixz="0.0"
-        iyy="${mass / 12.0 * (height3*height3 + width*width)}" iyz="0.0"
-        izz="${mass / 12.0 * (width*width + width*width)}"/>
+        ixx="0.3345833333333" ixy="0.0" ixz="0.0"
+        iyy="0.3345833333333" iyz="0.0"
+        izz="0.0025"/>
     </inertial>
   </link>

Commit message: change initial conditions and foot size/mass

File: double_pendulum_description/urdf/double_pendulum.xacro (robot description, xacro)
@@ -10,5 +10,6 @@
   <xacro:property name="height3" value="1.1" /> <!-- Link 3 -->
   <xacro:property name="foot_height" value="0.05" /> <!-- Foot dimensions -->
-  <xacro:property name="foot_width" value="0.5" />
+  <xacro:property name="foot_width" value="1.0" />
+  <xacro:property name="foot_mass" value="0.2" /> <!-- negligible mass for the foot -->
   <xacro:property name="axel_offset" value="0.05" /> <!-- How far keep joints away from each other -->
   <!-- Import all Gazebo-customization elements, including Gazebo colors -->
@@ -17,9 +18,10 @@
   <xacro:include filename="$(find double_pendulum_description)/urdf/materials.xacro" />
   <!-- Used for fixing robot foot to the world -->
+  <!--
   <link name="world"/>
   <joint name="fixed" type="fixed">
     <parent link="world"/>
     <child link="foot"/>
-  </joint>
+  </joint>-->
   <!-- Foot Link-->
   <link name="foot">
@@ -39,9 +41,9 @@
     <inertial>
       <origin xyz="0 0 ${foot_height/2}" rpy="0 0 0"/>
-      <mass value="${mass}"/>
+      <mass value="${foot_mass}"/>
     <inertia
-        ixx="${mass / 12.0 * (foot_width*foot_width + foot_height*foot_height)}" ixy="0.0" ixz="0.0"
-        iyy="${mass / 12.0 * (foot_height*foot_height + foot_width*foot_width)}" iyz="0.0"
-        izz="${mass / 12.0 * (foot_width*foot_width + foot_width*foot_width)}"/>
+        ixx="${foot_mass / 12.0 * (foot_width*foot_width + foot_height*foot_height)}" ixy="0.0" ixz="0.0"
+        iyy="${foot_mass / 12.0 * (foot_height*foot_height + foot_width*foot_width)}" iyz="0.0"
+        izz="${foot_mass / 12.0 * (foot_width*foot_width + foot_width*foot_width)}"/>
     </inertial>
   </link>
@@ -69,9 +71,9 @@
     <inertial>
       <origin xyz="0 0 ${height1/2}" rpy="0 0 0"/>
-      <mass value="${mass}"/>
+      <mass value="${foot_mass}"/>
     <inertia
-        ixx="${mass / 12.0 * (width*width + height1*height1)}" ixy="0.0" ixz="0.0"
-        iyy="${mass / 12.0 * (height1*height1 + width*width)}" iyz="0.0"
-        izz="${mass / 12.0 * (width*width + width*width)}"/>
+        ixx="${foot_mass / 12.0 * (width*width + height1*height1)}" ixy="0.0" ixz="0.0"
+        iyy="${foot_mass / 12.0 * (height1*height1 + width*width)}" iyz="0.0"
+        izz="${foot_mass / 12.0 * (width*width + width*width)}"/>
     </inertial>
   </link>

Commit message: revert to original inertia parameterization

File: double_pendulum_description/urdf/double_pendulum.xacro (robot description, xacro)
@@ -83,5 +83,5 @@
     <origin xyz="0 ${width} ${height1 - axel_offset}" rpy="0 0 0"/>
     <axis xyz="0 1 0"/>
-    <dynamics damping="0.5"/>
+    <dynamics damping="0.7"/>
   </joint>
   <!-- Middle Link -->
@@ -103,10 +103,9 @@
       <origin xyz="0 0 ${height2/2 - axel_offset}" rpy="0 0 0"/>
       <mass value="${mass}"/>
-      <!-- inertias copied from matlab model-->
       <inertia
-        ixx="0.3345833333333" ixy="0.0" ixz="0.0"
-        iyy="0.3345833333333" iyz="0.0"
-        izz="0.0025"/>
-    </inertial>
+          ixx="${mass / 12.0 * (width*width + height2*height2)}" ixy="0.0" ixz="0.0"
+          iyy="${mass / 12.0 * (height2*height2 + width*width)}" iyz="0.0"
+          izz="${mass / 12.0 * (width*width + width*width)}"/>
+      </inertial>
   </link>
   <joint name="joint2" type="continuous">
@@ -115,5 +114,5 @@
     <origin xyz="0 ${width} ${height2 - axel_offset*2}" rpy="0 0 0"/>
     <axis xyz="0 1 0"/>
-    <dynamics damping="0.5"/>
+    <dynamics damping="0.7"/>
   </joint>
   <!-- Top Link -->
@@ -136,8 +135,8 @@
       <mass value="${mass}"/>
       <inertia
-        ixx="0.3345833333333" ixy="0.0" ixz="0.0"
-        iyy="0.3345833333333" iyz="0.0"
-        izz="0.0025"/>
-    </inertial>
+          ixx="${mass / 12.0 * (width*width + height3*height3)}" ixy="0.0" ixz="0.0"
+          iyy="${mass / 12.0 * (height3*height3 + width*width)}" iyz="0.0"
+          izz="${mass / 12.0 * (width*width + width*width)}"/>
+      </inertial>
   </link>
   <!-- Motors so we can actuate the joints -->
